File: Mercury-v2-pcb.kicad_sch (KiCad schematic)
At the start: 0 parts

Commit message: feat: improve pcb
Changed lines of the file:
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@@
-	(wire
-		(pts
-			(xy 168.91 124.46) (xy 181.61 124.46)
-		)
-		(stroke
-			(width 0)
-			(type default)
-		)
-	)
 	(wire
 		(pts
@@
 	(wire
 		(pts
+			(xy 168.91 120.65) (xy 181.61 120.65)
+		)
+		(stroke
+			(width 0)
+			(type default)
+		)
+	)
+	(wire
+		(pts
 			(xy 109.22 139.7) (xy 127 139.7)
 		)
@@
 	(wire
 		(pts
-			(xy 168.91 120.65) (xy 181.61 120.65)
+			(xy 168.91 137.16) (xy 181.61 137.16)
 		)
 		(stroke
@@
 	(wire
 		(pts
+			(xy 168.91 133.35) (xy 181.61 133.35)
+		)
+		(stroke
+			(width 0)
+			(type default)
+		)
+	)
+	(wire
+		(pts
 			(xy 168.91 62.23) (xy 181.61 62.23)
-		)
-		(stroke
-			(width 0)
-			(type default)
-		)
-	)
-	(wire
-		(pts
-			(xy 168.91 137.16) (xy 181.61 137.16)
 		)
 		(stroke
@@
 		)
 		(pin "IR_LED2" input
-			(at 168.91 124.46 0)
+			(at 168.91 133.35 0)
 			(effects
 				(font
@@
 	)
 	(sheet
-		(at 181.61 118.11)
+		(at 181.61 130.81)
 		(size 24.13 8.89)
 		(fields_autoplaced yes)
@@
 		)
 		(property "Sheetname" "ir_led"
-			(at 181.61 117.3984 0)
+			(at 181.61 130.0984 0)
 			(effects
 				(font
@@
 		)
 		(property "Sheetfile" "ir_led.kicad_sch"
-			(at 181.61 127.5846 0)
+			(at 181.61 140.2846 0)
 			(effects
 				(font
@@
 		)
 		(pin "IR_LED_IN1" input
-			(at 181.61 120.65 180)
+			(at 181.61 133.35 180)
 			(effects
 				(font
@@
 		)
 		(pin "IR_LED_IN2" input
-			(at 181.61 124.46 180)
+			(at 181.61 137.16 180)
 			(effects
 				(font
@@
 	)
 	(sheet
-		(at 181.61 133.35)
+		(at 184.15 116.84)
 		(size 24.13 7.62)
 		(fields_autoplaced yes)
@@
 		)
 		(property "Sheetname" "ir_led_single"
-			(at 181.61 132.6384 0)
+			(at 184.15 116.1284 0)
 			(effects
 				(font
@@
 		)
 		(property "Sheetfile" "ir_led_single.kicad_sch"
-			(at 181.61 141.5546 0)
+			(at 184.15 125.0446 0)
 			(effects
 				(font
@@
 		)
 		(pin "IR_LED_IN" input
-			(at 181.61 137.16 180)
-			(effects
-				(font
-					(size 1.27 1.27)
-				)
-				(justify left)
-			)
-		)
+			(at 208.28 120.65 0)
+			(effects
+				(font
+					(size 1.27 1.27)
+				)
+				(justify right)
+			)
+		)

Commit message: feat: route tracks
Changed lines of the file:
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@@
 	)
 	(sheet
-		(at 184.15 116.84)
+		(at 181.61 116.84)
 		(size 24.13 7.62)
 		(fields_autoplaced yes)
@@
 		)
 		(property "Sheetname" "ir_led_single"
-			(at 184.15 116.1284 0)
+			(at 181.61 116.1284 0)
 			(effects
 				(font
@@
 		)
 		(property "Sheetfile" "ir_led_single.kicad_sch"
-			(at 184.15 125.0446 0)
+			(at 181.61 125.0446 0)
 			(effects
 				(font
@@
 		)
 		(pin "IR_LED_IN" input
-			(at 208.28 120.65 0)
+			(at 181.61 120.65 180)
 			(effects
 				(font
 					(size 1.27 1.27)
 				)
-				(justify right)
+				(justify left)
 			)
 		)
