File: ir_sensor.kicad_sch (KiCad schematic)
At the start: 11 parts, among them U2 AD8602

Commit message: feat: route tracks
Connections:
- net at D12.2, R20.1: now also C15.2; no longer C13.2
- net at D13.2, R22.1: now also C13.2; no longer C15.2
Other:
- moved on the sheet: D12, D13, R20, R22
Changed lines of the file:
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@@
+	)
+	(junction
+		(at 92.71 104.14)
+		(diameter 0)
+		(color 0 0 0 0)
 	)
 	(junction
@@
 	)
 	(junction
-		(at 173.99 104.14)
-		(diameter 0)
-		(color 0 0 0 0)
-	)
-	(junction
 		(at 210.82 87.63)
 		(diameter 0)
@@
 	)
 	(junction
-		(at 92.71 104.14)
+		(at 173.99 104.14)
 		(diameter 0)
 		(color 0 0 0 0)
@@
 	(wire
 		(pts
+			(xy 173.99 99.06) (xy 173.99 104.14)
+		)
+		(stroke
+			(width 0)
+			(type default)
+		)
+	)
+	(wire
+		(pts
 			(xy 190.5 87.63) (xy 198.12 87.63)
 		)
@@
 	(wire
 		(pts
+			(xy 92.71 87.63) (xy 92.71 91.44)
+		)
+		(stroke
+			(width 0)
+			(type default)
+		)
+	)
+	(wire
+		(pts
 			(xy 210.82 87.63) (xy 203.2 87.63)
 		)
@@
 	(wire
 		(pts
+			(xy 92.71 104.14) (xy 92.71 107.95)
+		)
+		(stroke
+			(width 0)
+			(type default)
+		)
+	)
+	(wire
+		(pts
 			(xy 105.41 104.14) (xy 109.22 104.14)
 		)
@@
 		)
 	)
+	(wire
+		(pts
+			(xy 92.71 99.06) (xy 92.71 104.14)
+		)
+		(stroke
+			(width 0)
+			(type default)
+		)
+	)
 	(polyline
 		(pts
@@
 	(wire
 		(pts
-			(xy 173.99 104.14) (xy 173.99 99.06)
-		)
-		(stroke
-			(width 0)
-			(type default)
-		)
-	)
-	(wire
-		(pts
 			(xy 210.82 101.6) (xy 215.9 101.6)
 		)
@@
 	(wire
 		(pts
-			(xy 92.71 118.11) (xy 92.71 114.3)
-		)
-		(stroke
-			(width 0)
-			(type default)
-		)
-	)
-	(wire
-		(pts
 			(xy 190.5 87.63) (xy 190.5 104.14)
 		)
@@
 	(wire
 		(pts
+			(xy 173.99 113.03) (xy 173.99 118.11)
+		)
+		(stroke
+			(width 0)
+			(type default)
+		)
+	)
+	(wire
+		(pts
 			(xy 109.22 78.74) (xy 109.22 87.63)
 		)
@@
 	(wire
 		(pts
-			(xy 173.99 118.11) (xy 173.99 114.3)
-		)
-		(stroke
-			(width 0)
-			(type default)
-		)
-	)
-	(wire
-		(pts
-			(xy 92.71 91.44) (xy 92.71 87.63)
-		)
-		(stroke
-			(width 0)
-			(type default)
-		)
-	)
-	(wire
-		(pts
-			(xy 92.71 109.22) (xy 92.71 104.14)
-		)
-		(stroke
-			(width 0)
-			(type default)
-		)
-	)
-	(wire
-		(pts
 			(xy 186.69 104.14) (xy 190.5 104.14)
 		)
@@
 	(wire
 		(pts
+			(xy 173.99 104.14) (xy 173.99 107.95)
+		)
+		(stroke
+			(width 0)
+			(type default)
+		)
+	)
+	(wire
+		(pts
 			(xy 109.22 87.63) (xy 109.22 104.14)
 		)
@@
 	(wire
 		(pts
+			(xy 92.71 113.03) (xy 92.71 118.11)
+		)
+		(stroke
+			(width 0)
+			(type default)
+		)
+	)
+	(wire
+		(pts
 			(xy 127 101.6) (xy 129.54 101.6)
 		)
@@
 	(wire
 		(pts
+			(xy 173.99 87.63) (xy 173.99 91.44)
+		)
+		(stroke
+			(width 0)
+			(type default)
+		)
+	)
+	(wire
+		(pts
 			(xy 203.2 78.74) (xy 210.82 78.74)
 		)
@@
 	(wire
 		(pts
-			(xy 173.99 91.44) (xy 173.99 87.63)
-		)
-		(stroke
-			(width 0)
-			(type default)
-		)
-	)
-	(wire
-		(pts
-			(xy 92.71 104.14) (xy 92.71 99.06)
-		)
-		(stroke
-			(width 0)
-			(type default)
-		)
-	)
-	(wire
-		(pts
 			(xy 181.61 104.14) (xy 173.99 104.14)
-		)
-		(stroke
-			(width 0)
-			(type default)
-		)
-	)
-	(wire
-		(pts
-			(xy 173.99 109.22) (xy 173.99 104.14)
 		)
 		(stroke
@@
 	(symbol
 		(lib_id "My_Device:SFH213FA")
-		(at 96.52 95.25 270)
+		(at 177.8 95.25 270)
 		(unit 1)
 		(exclude_from_sim no)
@@
 		(dnp no)
 		(property "Reference" "D12"
-			(at 80.01 93.98 90)
+			(at 161.29 93.98 90)
 			(effects
 				(font
@@
 		)
 		(property "Value" "SFH213FA"
-			(at 80.01 96.52 90)
+			(at 161.29 96.52 90)
 			(effects
 				(font
@@
 		)
 		(property "Footprint" "Diode_THT:D_T-1_P2.54mm_Vertical_AnodeUp"
-			(at 97.79 95.25 0)
+			(at 179.07 95.25 0)
 			(effects
 				(font
@@
 		)
 		(property "Datasheet" ""
-			(at 97.79 95.25 0)
+			(at 179.07 95.25 0)
 			(effects
 				(font
@@
 		)
 		(property "Description" ""
-			(at 96.52 95.25 0)
+			(at 177.8 95.25 0)
 			(effects
 				(font
@@
 	(symbol
 		(lib_id "My_Device:SFH213FA")
-		(at 177.8 95.25 270)
+		(at 96.52 95.25 270)
 		(unit 1)
 		(exclude_from_sim no)
@@
 		(dnp no)
 		(property "Reference" "D13"
-			(at 161.29 93.98 90)
+			(at 80.01 93.98 90)
 			(effects
 				(font
@@
 		)
 		(property "Value" "SFH213FA"
-			(at 161.29 96.52 90)
+			(at 80.01 96.52 90)
 			(effects
 				(font
@@
 		)
 		(property "Footprint" "Diode_THT:D_T-1_P2.54mm_Vertical_AnodeUp"
-			(at 179.07 95.25 0)
+			(at 97.79 95.25 0)
 			(effects
 				(font
@@
 		)
 		(property "Datasheet" ""
-			(at 179.07 95.25 0)
+			(at 97.79 95.25 0)
 			(effects
 				(font
@@
 		)
 		(property "Description" ""
-			(at 177.8 95.25 0)
+			(at 96.52 95.25 0)
 			(effects
 				(font
@@
 	(symbol
 		(lib_id "Device:R_Small")
-		(at 92.71 111.76 0)
+		(at 173.99 110.49 0)
 		(unit 1)
 		(exclude_from_sim no)
@@
 		(dnp no)
 		(property "Reference" "R20"
-			(at 94.2086 110.5916 0)
+			(at 175.4886 109.3216 0)
 			(effects
 				(font
@@
 		)
 		(property "Value" "100k"
-			(at 94.2086 112.903 0)
+			(at 175.4886 111.633 0)
 			(effects
 				(font
@@
 		)
 		(property "Footprint" "Resistor_SMD:R_0603_1608Metric"
-			(at 92.71 111.76 0)
+			(at 173.99 110.49 0)
 			(effects
 				(font
@@
 		)
 		(property "Datasheet" "~"
-			(at 92.71 111.76 0)
+			(at 173.99 110.49 0)
 			(effects
 				(font
@@
 		)
 		(property "Description" ""
-			(at 92.71 111.76 0)
+			(at 173.99 110.49 0)
 			(effects
 				(font
@@
 	(symbol
 		(lib_id "Device:R_Small")
-		(at 173.99 111.76 0)
+		(at 92.71 110.49 0)
 		(unit 1)
 		(exclude_from_sim no)
@@
 		(dnp no)
 		(property "Reference" "R22"
-			(at 175.4886 110.5916 0)
+			(at 94.2086 109.3216 0)
 			(effects
 				(font
@@
 		)
 		(property "Value" "100k"
-			(at 175.4886 112.903 0)
+			(at 94.2086 111.633 0)
 			(effects
 				(font
@@
 		)
 		(property "Footprint" "Resistor_SMD:R_0603_1608Metric"
-			(at 173.99 111.76 0)
+			(at 92.71 110.49 0)
 			(effects
 				(font
@@
 		)
 		(property "Datasheet" "~"
-			(at 173.99 111.76 0)
+			(at 92.71 110.49 0)
 			(effects
 				(font
@@
 		)
 		(property "Description" ""
-			(at 173.99 111.76 0)
-			(effects
-				(font
+			(at 92.71 110.49 0)
+			(effects
+				(font
